File: Button-PCB.sch (KiCad schematic (older format))
At the start: 32 parts

Commit message: Initial part annotation
Parts:
- gave numbers to parts that had none: 32

Commit message: Assigning footprints for resistors (0805), caps (0805) and buffer (SOIC-N)
Parts:
- C1, C2, C3: footprint (none) -> Capacitors_SMD:C_0805
- R1, R10, R11, R12, R13, R2, R3, R4, R5, R6, R7, R8, R9: footprint (none) -> Resistors_SMD:R_0805
- U1: footprint (none) -> TO_SOT_Packages_SMD:SOT-223-3Lead_TabPin2

Commit message: Swap out FDS4435BZ symbol with one of the correct pinout for the SOIC-8 footprint.
Parts:
- removed Q1: FDS4435BZ, symbol Q_PMOS_SDG
- added Q1: FDS4435BZ, SMD_Packages:SOIC-8-N, symbol IRF7606PBF
- U2: footprint (none) -> SMD_Packages:SOIC-14_N
Connections:
- net GND: now also Q1.4 (G)
- net VPP: now also Q1.1 (S), Q1.2 (S), Q1.3 (S)
- net at J8.2 (P2): now also Q1.5 (D), Q1.6 (D), Q1.7 (D), Q1.8 (D)
Other:
- note added: "Reverse Polarity Protection"
- note removed: "Reverse Polarity Protection\nP-FET to use: FDS4435BZ"
- note removed: "Take care, special package"

Commit message: Adding GND pin to UART and RES connectors.
Parts:
- J2: symbol CONN_01X02 -> CONN_01X03
- J5: symbol CONN_01X03 -> CONN_01X04
Connections:
- net GND: now also J2.3 (P3), J5.4 (P4)
Changed lines of the file:
@@
 Button Input
 $Comp
-L CONN_01X02 J2
+L CONN_01X03 J2
 U 1 1 593F43D5
-P 6200 950
-F 0 "J2" H 6200 1100 50  0000 C CNN
-F 1 "UART" V 6300 950 50  0000 C CNN
-F 2 "" H 6200 950 50  0001 C CNN
-F 3 "" H 6200 950 50  0001 C CNN
-	1    6200 950
-	1    0    0    -1
-$EndComp
-$Comp
-L CONN_01X03 J5
+P 6200 1000
+F 0 "J2" H 6200 1200 50  0000 C CNN
+F 1 "UART" V 6300 1000 50  0000 C CNN
+F 2 "" H 6200 1000 50  0001 C CNN
+F 3 "" H 6200 1000 50  0001 C CNN
+	1    6200 1000
+	1    0    0    -1
+$EndComp
+$Comp
+L CONN_01X04 J5
 U 1 1 593F4607
-P 6200 1400
-F 0 "J5" H 6200 1600 50  0000 C CNN
-F 1 "RES" V 6300 1400 50  0000 C CNN
-F 2 "" H 6200 1400 50  0001 C CNN
-F 3 "" H 6200 1400 50  0001 C CNN
-	1    6200 1400
+P 6200 1550
+F 0 "J5" H 6200 1800 50  0000 C CNN
+F 1 "RES" V 6300 1550 50  0000 C CNN
+F 2 "" H 6200 1550 50  0001 C CNN
+F 3 "" H 6200 1550 50  0001 C CNN
+	1    6200 1550
 	1    0    0    -1
 $EndComp
@@
 Text Label 5900 1000 2    60   ~ 0
 RX
-Text Label 5900 1300 2    60   ~ 0
+Text Label 5900 1400 2    60   ~ 0
 H1
-Text Label 5900 1400 2    60   ~ 0
+Text Label 5900 1500 2    60   ~ 0
 H2
-Text Label 5900 1500 2    60   ~ 0
+Text Label 5900 1600 2    60   ~ 0
 H3
 $Comp
@@
 	6550 2500 6550 550
 Wire Wire Line
-	5900 1300 6000 1300
-Wire Wire Line
-	6000 1400 5900 1400
+	5900 1400 6000 1400
 Wire Wire Line
 	6000 1500 5900 1500
+Wire Wire Line
+	6000 1600 5900 1600
 Wire Wire Line
 	6000 900  5900 900
@@
 	1250 1750 1150 1750
 Connection ~ 1150 1750
+$Comp
+L GND #PWR?
+U 1 1 5945DAFF
+P 5900 1750
+F 0 "#PWR?" H 5900 1500 50  0001 C CNN
+F 1 "GND" H 5900 1600 50  0000 C CNN
+F 2 "" H 5900 1750 50  0001 C CNN
+F 3 "" H 5900 1750 50  0001 C CNN
+	1    5900 1750
+	1    0    0    -1
+$EndComp
+$Comp
+L GND #PWR?
+U 1 1 5945DB85
+P 5900 1150
+F 0 "#PWR?" H 5900 900 50  0001 C CNN
+F 1 "GND" H 5900 1000 50  0000 C CNN
+F 2 "" H 5900 1150 50  0001 C CNN
+F 3 "" H 5900 1150 50  0001 C CNN
+	1    5900 1150
+	1    0    0    -1
+$EndComp
+Wire Wire Line
+	6000 1700 5900 1700
+Wire Wire Line
+	5900 1700 5900 1750
+Wire Wire Line
+	6000 1100 5900 1100
+Wire Wire Line
+	5900 1100 5900 1150
 $EndSCHEMATC

Commit message: Using standard 2.54" headers for all connectors for now. Will change later.
Parts:
- J1, J11, J6, J7, J8, JP1: footprint (none) -> Pin_Headers:Pin_Header_Straight_1x02_Pitch2.54mm
- J10, J3, J4, J9: footprint (none) -> Pin_Headers:Pin_Header_Angled_1x03_Pitch2.54mm
- J2: footprint (none) -> Pin_Headers:Pin_Header_Straight_1x03_Pitch2.54mm
- J5: footprint (none) -> Pin_Headers:Pin_Header_Straight_1x04_Pitch2.54mm
Changed lines of the file:
@@
 F 0 "J8" H 800 2000 50  0000 C CNN
 F 1 "Power IN" V 900 1850 50  0000 C CNN
-F 2 "" H 800 1850 50  0001 C CNN
+F 2 "Pin_Headers:Pin_Header_Straight_1x02_Pitch2.54mm" H 800 1850 50  0001 C CNN
 F 3 "" H 800 1850 50  0001 C CNN
 	1    800  1850
@@
 F 0 "J9" H 9350 2150 50  0000 C CNN
 F 1 "Strip 2" V 9450 1950 50  0000 C CNN
-F 2 "" H 9350 1950 50  0001 C CNN
+F 2 "Pin_Headers:Pin_Header_Angled_1x03_Pitch2.54mm" H 9350 1950 50  0001 C CNN
 F 3 "" H 9350 1950 50  0001 C CNN
 	1    9350 1950
@@
 F 0 "J3" H 9350 1350 50  0000 C CNN
 F 1 "Strip 1" V 9450 1150 50  0000 C CNN
-F 2 "" H 9350 1150 50  0001 C CNN
+F 2 "Pin_Headers:Pin_Header_Angled_1x03_Pitch2.54mm" H 9350 1150 50  0001 C CNN
 F 3 "" H 9350 1150 50  0001 C CNN
 	1    9350 1150
@@
 F 0 "J7" H 7750 1750 50  0000 C CNN
 F 1 "Button" V 7850 1600 50  0000 C CNN
-F 2 "" H 7750 1600 50  0001 C CNN
+F 2 "Pin_Headers:Pin_Header_Straight_1x02_Pitch2.54mm" H 7750 1600 50  0001 C CNN
 F 3 "" H 7750 1600 50  0001 C CNN
 	1    7750 1600
@@
 F 0 "J10" H 10850 2150 50  0000 C CNN
 F 1 "Strip 4" V 10950 1950 50  0000 C CNN
-F 2 "" H 10850 1950 50  0001 C CNN
+F 2 "Pin_Headers:Pin_Header_Angled_1x03_Pitch2.54mm" H 10850 1950 50  0001 C CNN
 F 3 "" H 10850 1950 50  0001 C CNN
 	1    10850 1950
@@
 F 0 "J4" H 10850 1350 50  0000 C CNN
 F 1 "Strip 3" V 10950 1150 50  0000 C CNN
-F 2 "" H 10850 1150 50  0001 C CNN
+F 2 "Pin_Headers:Pin_Header_Angled_1x03_Pitch2.54mm" H 10850 1150 50  0001 C CNN
 F 3 "" H 10850 1150 50  0001 C CNN
 	1    10850 1150
@@
 F 0 "J2" H 6200 1200 50  0000 C CNN
 F 1 "UART" V 6300 1000 50  0000 C CNN
-F 2 "" H 6200 1000 50  0001 C CNN
+F 2 "Pin_Headers:Pin_Header_Straight_1x03_Pitch2.54mm" H 6200 1000 50  0001 C CNN
 F 3 "" H 6200 1000 50  0001 C CNN
 	1    6200 1000
@@
 F 0 "J5" H 6200 1800 50  0000 C CNN
 F 1 "RES" V 6300 1550 50  0000 C CNN
-F 2 "" H 6200 1550 50  0001 C CNN
+F 2 "Pin_Headers:Pin_Header_Straight_1x04_Pitch2.54mm" H 6200 1550 50  0001 C CNN
 F 3 "" H 6200 1550 50  0001 C CNN
 	1    6200 1550
@@
 F 0 "J6" H 5450 1700 50  0000 C CNN
 F 1 "5V" V 5550 1550 50  0000 C CNN
-F 2 "" H 5450 1550 50  0001 C CNN
+F 2 "Pin_Headers:Pin_Header_Straight_1x02_Pitch2.54mm" H 5450 1550 50  0001 C CNN
 F 3 "" H 5450 1550 50  0001 C CNN
 	1    5450 1550
@@
 F 0 "J11" H 5450 2300 50  0000 C CNN
 F 1 "3V3" V 5550 2150 50  0000 C CNN
-F 2 "" H 5450 2150 50  0001 C CNN
+F 2 "Pin_Headers:Pin_Header_Straight_1x02_Pitch2.54mm" H 5450 2150 50  0001 C CNN
 F 3 "" H 5450 2150 50  0001 C CNN
 	1    5450 2150
@@
 F 0 "J1" H 5450 1100 50  0000 C CNN
 F 1 "VPP" V 5550 950 50  0000 C CNN
-F 2 "" H 5450 950 50  0001 C CNN
+F 2 "Pin_Headers:Pin_Header_Straight_1x02_Pitch2.54mm" H 5450 950 50  0001 C CNN
 F 3 "" H 5450 950 50  0001 C CNN
 	1    5450 950
@@
 F 0 "JP1" H 3450 1050 50  0000 C CNN
 F 1 "Reg Bypass" H 3450 820 50  0000 C CNN
-F 2 "" H 3450 900 50  0001 C CNN
+F 2 "Pin_Headers:Pin_Header_Straight_1x02_Pitch2.54mm" H 3450 900 50  0001 C CNN
 F 3 "" H 3450 900 50  0001 C CNN
 	1    3450 900
@@
 Connection ~ 1150 1750
 $Comp
-L GND #PWR?
+L GND #PWR036
 U 1 1 5945DAFF
 P 5900 1750
-F 0 "#PWR?" H 5900 1500 50  0001 C CNN
+F 0 "#PWR036" H 5900 1500 50  0001 C CNN
 F 1 "GND" H 5900 1600 50  0000 C CNN
 F 2 "" H 5900 1750 50  0001 C CNN
@@
 $EndComp
 $Comp
-L GND #PWR?
+L GND #PWR037
 U 1 1 5945DB85
 P 5900 1150
-F 0 "#PWR?" H 5900 900 50  0001 C CNN
+F 0 "#PWR037" H 5900 900 50  0001 C CNN
 F 1 "GND" H 5900 1000 50  0000 C CNN
 F 2 "" H 5900 1150 50  0001 C CNN

Commit message: Assigning NodeMCU footprint
Parts:
- U3: footprint (none) -> nodemcuv3:nodemcu_v3
Changed lines of the file:
@@
 F 0 "U3" H 3200 7300 60  0000 C CNN
 F 1 "NodeMCUv3" H 2650 7300 60  0000 C CNN
-F 2 "" H 2900 6150 60  0001 C CNN
+F 2 "nodemcuv3:nodemcu_v3" H 2900 6150 60  0001 C CNN
 F 3 "" H 2900 6150 60  0001 C CNN
 	1    2900 6150
