File: Button-PCB.kicad_pcb (KiCad board)
At the start: 2 copper layers, 50 x 50 mm, 32 parts, among them J1 VPP, J10 Strip 3, J11 3V3, J2 UART, J3 Strip 1, J4 Strip 4, J5 RES, J7 Button, J8 Power IN, J9 Strip 2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

Commit message: hacking bugs
Parts:
- moved U3 16.6 mm to (30.8, 43.5)
- moved R5 4.72 mm to (27.5, 54.3)
- moved R6 4.63 mm to (27.5, 62.5)
- moved R2 4.50 mm to (27.5, 57.9)
- moved R1 1.34 mm to (27.5, 51.3), turned to 180 degrees
Routing:
- net GND: track 278.5 -> 209.5 mm
- net +3V3: track 23.5 -> 74.4 mm, vias 0 -> 1
- net Net-(R11-Pad2): track 6.59 -> 14.9 mm
- net Net-(R12-Pad2): track 7.39 -> 12.7 mm
- net Net-(R10-Pad2): track 6.53 -> 11.9 mm
- net Net-(U3-Pad30): track 0.00 -> 5.08 mm
- net Net-(U3-Pad27): track 0.00 -> 5.08 mm
- net /BUT_1: track 11.7 -> 16.2 mm
- net /TX: track 19.5 -> 20.6 mm
- added copper zone on B.Cu, net GND
Other:
- board text added: "+"
- board text added: "-"
- board text added: "Bat"
- board text added: "Buf1"
- board text added: "Buf2"
- board text added: "Buf3"
- board text added: "Buf4"
- board text added: "Button1"
